File: MiniJoystickMiniStepper/MiniJoyMiniStepper.sch (KiCad schematic (older format))
At the start: 21 parts, among them J1 STEPPER_UNI_5P, J10 TH_0.1_1x1, J11 TH_0.1_1x1, J2 STEPPER_UNI_5P, J28 TH_0.1_1x1, J29 TH_0.1_1x1, J50 STEPPER_UNI_5P, J51 STEPPER_UNI_5P, J6 TH_0.1_1x1, J7 TH_0.1_1x1, J8 TH_0.1_1x1, J9 TH_0.1_1x1, U1 ADAFRUIT_FEATHER_M0

Commit message: More routing. 68 nets left.
Parts:
- gave numbers to parts that had none: 2
Changed lines of the file:
@@
 Text Label 6700 1000 0    39   ~ 0
 M3_C3
+Text Label 4400 5450 0    39   ~ 0
+M2_C0
 Text Label 4400 5350 0    39   ~ 0
-M2_C0
-Text Label 4400 5450 0    39   ~ 0
 M2_C1
 Text Label 6900 4950 0    39   ~ 0
@@
 	6600 1000 7200 1000
 Wire Wire Line
+	4300 5450 4900 5450
+Wire Wire Line
 	4300 5350 4900 5350
-Wire Wire Line
-	4300 5450 4900 5450
 Wire Wire Line
 	6800 4950 7400 4950
@@
 	8700 1950 9300 1950
 $Comp
-L ULN2803 U?
+L ULN2803 U2
 U 1 1 586C241A
 P 9500 1850
-F 0 "U?" H 9350 3000 60  0000 C CNN
+F 0 "U2" H 9350 3000 60  0000 C CNN
 F 1 "ULN2803" H 9550 350 60  0000 C CNN
 F 2 "" H 9550 2200 60  0001 C CNN
@@
 $EndComp
 $Comp
-L ULN2803 U?
+L ULN2803 U3
 U 1 1 586C2749
 P 9500 4650
-F 0 "U?" H 9350 5800 60  0000 C CNN
+F 0 "U3" H 9350 5800 60  0000 C CNN
 F 1 "ULN2803" H 9550 3150 60  0000 C CNN
 F 2 "" H 9550 5000 60  0001 C CNN
