File: MiniJoystickMiniStepper/MiniJoyMiniStepper.kicad_pcb (KiCad board)
At the start: 2 copper layers, 21 parts, among them J1 STEPPER_UNI_5P, J10 TH_0.1_1x1, J11 TH_0.1_1x1, J2 STEPPER_UNI_5P, J28 TH_0.1_1x1, J29 TH_0.1_1x1, J50 STEPPER_UNI_5P, J51 STEPPER_UNI_5P, J6 TH_0.1_1x1, J7 TH_0.1_1x1, J8 TH_0.1_1x1, J9 TH_0.1_1x1, U1 ADAFRUIT_FEATHER_M0, U2 ULN2803, U3 ULN2803

Commit message: More routing. 68 nets left.
Parts:
- moved VCC1 94.4 mm to (114.3, 73.7)
- moved COM0 93.4 mm to (114.3, 76.2)
- moved GND1 92.5 mm to (114.3, 78.7)
- moved SHIELD1 88.9 mm to (132.1, 63.5), turned to 270 degrees
- moved J8 78.5 mm to (111.5, 91.9)
- moved J29 76.1 mm to (208.3, 91.4)
- moved J28 69.5 mm to (208.3, 119.4)
- moved J7 67.3 mm to (124.5, 116.8)
- moved J10 66.5 mm to (124.5, 121.9)
- moved J9 63.6 mm to (124.5, 119.4)
- moved J6 62.9 mm to (124.5, 114.3)
- moved J11 60.7 mm to (111.8, 109.7)
- moved U1 41.0 mm to (149.9, 114.3), turned to 270 degrees
- moved R2 40.3 mm to (111.6, 117.9)
- moved R1 6.87 mm to (111.6, 100.1)
Connections:
- SHIELD1 pad AD4: /M2_C0 -> /M2_C1
- SHIELD1 pad AD5: /M2_C1 -> /M2_C0
Routing:
- net GND: track 8.77 -> 141.2 mm
- net VCC: track 0.00 -> 108.2 mm
- net /JOY0_AXIS0: track 0.00 -> 73.8 mm
- net /JOY1_AXIS0: track 0.00 -> 66.8 mm
- net /JOY0_AXIS1: track 0.00 -> 63.3 mm
- net /M2_C2: track 68.5 -> 6.51 mm, vias 1 -> 0
- net /JOY1_AXIS1: track 0.00 -> 60.6 mm
- net /M2_C1: track 40.0 -> 98.0 mm
- net /M2_C0: track 43.9 -> 98.3 mm
- net /M2_C3: track 33.3 -> 5.99 mm
- net /M0_C2: track 6.51 -> 31.7 mm
- net /M0_C3: track 5.99 -> 26.1 mm
- net /M0_C1: track 7.04 -> 27.1 mm
- net /M0_C0: track 7.75 -> 27.8 mm
- net /M1_C0: track 5.46 -> 25.6 mm
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
Commit message: Finalized board. Ready for proto fab.
Routing:
- net VCC: track 108.2 -> 314.9 mm, vias 0 -> 2
- net /COM: track 53.0 -> 227.5 mm, vias 0 -> 1
- net GND: track 141.2 -> 290.5 mm
- net /M2_C2: track 6.51 -> 114.4 mm, vias 0 -> 1
- net /M3_C3: track 7.04 -> 114.7 mm, vias 0 -> 2
- net /M3_C2: track 6.51 -> 112.4 mm, vias 0 -> 1
- net /M3_C0: track 5.46 -> 103.0 mm, vias 0 -> 1
- net /M2_C3: track 5.99 -> 68.2 mm, vias 0 -> 1
- net /M3_C1: track 25.4 -> 72.6 mm
- net /M1_C3: track 14.2 -> 57.0 mm
- net /M2_C0: track 98.3 -> 108.3 mm
- net /M1_C2: track 23.9 -> 31.5 mm
- net /M0_C0: track 27.8 -> 35.2 mm
- net /M1_C0: track 25.6 -> 32.9 mm
- net /M0_C3: track 26.1 -> 33.4 mm
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Other:
- board outline added: 127 x 73.7 mm
- board text added: "ADAFRUIT FEATHER"
- board text added: "Arduino Goes Here"
- board text added: "Believotron 4-Axis Motor 2 Joystick Adapter Board PCBBT-4CH-2XY-A0 2017-01-01 It was better next year"
- board text added: "CTS Electrocomponents 254TA103B50B"
- board text added: "These chips eat their spinach"
- board text added: "ULN2803"
